File: mts-demod/.history/mts-demod.kicad_sch (KiCad schematic)
At the start: 20 parts, among them U1 FDS010, U2 OPA858IDSGR

Commit message: completed stage two of TIA
Parts:
- added C11, C12, C13, C15: 10n, Capacitor_SMD:C_0402_1005Metric, symbol Device:C
- added C14: 0.1u, Capacitor_SMD:C_0402_1005Metric, symbol Device:C
- added R10, R11: 49.9, Resistor_SMD:R_0402_1005Metric, symbol Device:R
- added R6, R7: 1k, Capacitor_SMD:C_0603_1608Metric, symbol Device:R
- added R8: 348, Resistor_SMD:R_0402_1005Metric, symbol Device:R
- added R9: 49.9, Capacitor_SMD:C_0603_1608Metric, symbol Device:R
- added U3: OPA695IDR, D8, symbol OPA695:OPA695IDR
Connections:
- net +5VA: now also C13.1, C14.2, R6.2, U3.7 (VS+), U3.8 (*DIS)
- net GND: now also C12.1, C13.2, C14.1, R7.1, U3.4 (VS-)
- net 858_OUT: now reaches C10.2, TP1.1
- net 858_OUT: now also R6.1, R7.2, U3.3 (NONINVERTINGINPUT)
- new net: C15.1, R11.1
- new net: C11.1, R10.1
- new net: C12.2, R9.2
- new net 695_ADC_PATH: C11.2
- new net 695_MIXER_PATH: C15.2
- new net INV_695: R8.2, R9.1, U3.2 (INVERTINGINPUT)
- new net OUT_695: R10.2, R11.2, R8.1, U3.6 (OUTPUT)
- no-connect marks 1 -> 5
Other:
- note added: "TIA Stage 1 (1.24k ohms)"
- note added: "TIA Stage 2 (8 V/V)"
- note removed: "OPA858 TIA (stage 1)"

Commit message: almost done with demod sch
Parts:
- added C16: 1.5p, Capacitor_SMD:C_0402_1005Metric, symbol Device:C
- added C17: 1.5p, Mounting_Wuerth:Mounting_Wuerth_WA-SMSI-M2_H4mm_9774040243, symbol Device:C
- added C18, C19: 75p, Capacitor_SMD:C_0805_2012Metric, symbol Device:C
- added C20, C25: 2.4n, Capacitor_SMD:C_0402_1005Metric, symbol Device:C
- added C21, C23: 240p, Capacitor_SMD:C_0805_2012Metric, symbol Device:C
- added C22, C24: 110p, Capacitor_SMD:C_0805_2012Metric, symbol Device:C
- added C26: 0.1u, Capacitor_SMD:C_0402_1005Metric, symbol Device:C
- added C27: 470p, Capacitor_SMD:C_0805_2012Metric, symbol Device:C
- added C28: 620p, Capacitor_SMD:C_0805_2012Metric, symbol Device:C
- added IC1: ADE-1+, ADE1, symbol ADE-1+:ADE-1+
- added J1: RAW ERROR, SMA-J-P-H-ST-TH1:CONN_SMA-J-P-H-ST-TH1_SAI, symbol Connector:Conn_Coaxial
- added J2: DEMOD IN, SMA-J-P-H-ST-TH1:CONN_SMA-J-P-H-ST-TH1_SAI, symbol Connector:Conn_Coaxial
- added J3: DEMOD INPUT, SMA-J-P-H-ST-TH1:CONN_SMA-J-P-H-ST-TH1_SAI, symbol Connector:Conn_Coaxial
- added J4: DEMODED SIGNAL, SMA-J-P-H-ST-TH1:CONN_SMA-J-P-H-ST-TH1_SAI, symbol Connector:Conn_Coaxial
- added L1: 4.7u, Inductor_SMD:L_0603_1608Metric, symbol Device:L
- added L2: 680n, Inductor_SMD:L_0805_2012Metric, symbol Device:L
- added L3: 270n, symbol Device:L
- added L4, L5, L6, L7: 560n, Inductor_SMD:L_0805_2012Metric, symbol Device:L
- added R12: 296, Capacitor_SMD:C_0603_1608Metric, symbol Device:R
- added R13: 100, Capacitor_SMD:C_0603_1608Metric, symbol Device:R
- added U4: TCP-2-10X, RF_Mini-Circuits:Mini-Circuits_DB1627, symbol RF:TCP-2-10X
- added U5: GVA-81, Package_TO_SOT_SMD:SOT-89-3, symbol RF_Amplifier:GVA-81
- added U6: 0 dB atten, RF_Converter:RF_Attenuator_Susumu_PAT1220, symbol RF:PAT1220-C-0DB
- added U7: PAT1220-C-4DB, RF_Converter:RF_Attenuator_Susumu_PAT1220, symbol RF:PAT1220-C-4DB
- FB1: footprint (none) -> Inductor_SMD:L_0805_2012Metric
Connections:
- net +5VA: now also C26.1, L1.1
- net GND: now also C16.2, C17.2, C18.2, C19.2, C21.2, C22.2, C23.2, C24.2, C26.2, C27.1, C28.1, IC1.1 (GROUND_1), IC1.4 (GROUND_2), IC1.5 (GROUND_3), J1.2 (Ext), J2.2 (Ext), J3.2 (Ext), J4.2 (Ext), U4.1 (GND), U5.2 (GND), U6.3, U7.3
- net INV_695: now also R12.2
- net at C12.2, R9.2: now also R12.1
- net 695_ADC_PATH renamed 25MHz_LPF1
- net 25MHz_LPF1: now also C19.1, L6.1
- net 695_MIXER_PATH renamed 25MHz_LPF2
- net 25MHz_LPF2: now also C18.1, L4.1
- new net: C16.1, C17.1, U4.2 (CON), U4.5 (CON)
- new net: R13.1, U4.3 (PORT1), U6.1
- new net: C21.1, L4.2, L5.1
- new net: C28.2, L2.2, L3.1
- new net: C23.1, L6.2, L7.1
- new net: C20.1, U5.1
- new net: C25.2, L1.2, U5.3
- new net 10MHz_DEMOD_IN: J2.1 (In), U4.6 (SUM)
- new net 25MHz_LPF2_OUT: C22.1, IC1.3 (RF), L5.2
- new net ADC_CH0: C24.1, J1.1 (In), L7.2
- new net ADC_CH1: J3.1 (In), U6.2
- new net ADC_CH1b: J4.1 (In)
- new net DEMOD_LO: IC1.2 (IF), IC1.6 (LO), U7.2
- new net DEMOD_POSTAMP: C25.1, C27.2, L2.1
- new net DEMOD_POSTFILT: L3.2, U7.1
- new net DEMOD_PREAMP: C20.2, R13.2, U4.4 (PORT2)
- no-connect marks 5 -> 3
Other:
- note added: "(R12 is DNP, compensate 1.2 dB IL)"
- note added: "10 dB LO amplifier"
- note added: "25 MHz cleanup filters (5th order, Chebyshev)"
- note added: "Demod mixer"
- note added: "Input Splitter (0.5 dB IL)"
- note added: "LO post-amp cleanup"
- moved on the sheet: C12, R9

Commit message: demod sch is complete
Parts:
- removed C26: 0.1u, Capacitor_SMD:C_0402_1005Metric, symbol Device:C
- removed TP1: TIA1_COUP, symbol Connector:TestPoint
- added C29, C32, C35: 22u, Capacitor_SMD:C_0805_2012Metric, symbol Device:C
- added C30, C33, C36: 10u, Capacitor_SMD:C_0805_2012Metric, symbol Device:C
- added C31, C34, C38: 0.1u, Capacitor_SMD:C_0603_1608Metric, symbol Device:C
- added C37: 2.2u, Capacitor_SMD:C_0603_1608Metric, symbol Device:C
- added C39: 10n, Capacitor_SMD:C_0402_1005Metric, symbol Device:C
- added D1, D2, D3: LED, LED_SMD:LED_0603_1608Metric, symbol Device:LED
- added FB2: 1000 ohm, Inductor_SMD:L_0805_2012Metric, symbol Device:FerriteBead
- added J5: PLP-5+, PLP-5+:MINI-CIRCUITS_A01_CERN, symbol Connector_Generic_MountingPin:Conn_01x08_MountingPin
- added J6: INPUT PWR, CONN_SD-43045-005_08_MOL, symbol 430450812:430450812
- added R14: 1.5k, Capacitor_SMD:C_0603_1608Metric, symbol Device:R
- added R15: 3.3k, Capacitor_SMD:C_0603_1608Metric, symbol Device:R
- added R16: 5.6k, Capacitor_SMD:C_0603_1608Metric, symbol Device:R
- added U8: 6 dB pad, RF_Converter:RF_Attenuator_Susumu_PAT1220, symbol RF:PAT1220-C-4DB
- C1, C7, C8, R1: footprint (none) -> Capacitor_SMD:C_0603_1608Metric
- C10, C9: footprint (none) -> Capacitor_SMD:C_0402_1005Metric
- C14: footprint Capacitor_SMD:C_0402_1005Metric -> Capacitor_SMD:C_0603_1608Metric
- C5: value 0.22u -> 0.1u
- J4: value DEMODED SIGNAL -> ANALOG ERROR
- R2, R3, R4: footprint (none) -> Resistor_SMD:R_0603_1608Metric
- R5: footprint (none) -> Resistor_SMD:R_0402_1005Metric
Connections:
- net IN-_OPA858 is gone; now on net FDS010_ANODE: C9.1, R4.1, U2.3 (IN-)
- net +15V: now also C29.1, C30.1, C31.1, D3.2 (A), J6.3, J6.4
- net +5V: now also C35.1, C36.1, D1.2 (A), FB2.1, J6.7, J6.8
- net +5VA: no longer L1.1
- net 25MHz_LPF2_OUT: now also U8.1; no longer IC1.3 (RF)
- net ADC_CH1b: now also J5.8 (Pin_8)
- net DEMOD_LO: no longer IC1.2 (IF)
- net GND: now also C29.2, C30.2, C31.2, C32.2, C33.2, C34.2, C35.2, C36.2, C37.2, C38.2, C39.2, J5.2 (Pin_2), J5.3 (Pin_3), J5.4 (Pin_4), J5.5 (Pin_5), J5.6 (Pin_6), J5.7 (Pin_7), J6.5, J6.6, R14.2, R15.2, R16.2, U8.3
- net at R5.1, U2.6 (OUT): no longer TP2.1
- net at C10.1, R5.2: now also TP2.1
- new net: IC1.3 (RF), U8.2
- new net: D3.1 (K), R16.1
- new net: D2.1 (K), R15.1
- new net: D1.1 (K), R14.1
- new net +10V: C32.1, C33.1, C34.1, D2.2 (A), J6.1, J6.2
- new net +5VA_GVA: C37.1, C38.1, C39.1, FB2.2, L1.1
- new net DEMOD_IF: IC1.2 (IF), J5.1 (Pin_1)
- no-connect marks 3 -> 4
Other:
- note added: "+10V, +15V Power Supply"
- note added: "4 V/V per path"
- note added: "5 MHz, post-mixer"
- note added: "Input Splitter (0.5 dB excess IL)"
- note added: "Power Status LEDs"
- note removed: "Input Splitter (0.5 dB IL)"
- moved on the sheet: C16, C17, C20, C25, C27, C28, IC1, L1, L2, L3, R13, R5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

Commit message: init layout, pwr sections
Parts:
- added TP1: TestPoint, TestPoint:TestPoint_Keystone_5015_Micro_Mini, symbol Connector:TestPoint
- C17: footprint Mounting_Wuerth:Mounting_Wuerth_WA-SMSI-M2_H4mm_9774040243 -> Capacitor_SMD:C_0402_1005Metric
- IC1: footprint ADE1 -> ADE-1+:ADE1
- J6: footprint CONN_SD-43045-005_08_MOL -> 430450812:CONN_SD-43045-005_08_MOL
- L3: footprint (none) -> Inductor_SMD:L_0805_2012Metric
- TP2: footprint (none) -> TestPoint:TestPoint_Keystone_5015_Micro_Mini
- U2: footprint DSG0008A -> OPA858:DSG0008A
- U3: footprint D8 -> OPA695:D8
Connections:
- net +10V: now also TP1.1
Changed lines of the file:
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@@
 	)
 	(junction
+		(at 166.37 182.88)
+		(diameter 0)
+		(color 0 0 0 0)
+	)
+	(junction
 		(at 259.08 153.67)
 		(diameter 0)
@@
 			)
 		)
-		(property "Footprint" "Mounting_Wuerth:Mounting_Wuerth_WA-SMSI-M2_H4mm_9774040243"
+		(property "Footprint" "Capacitor_SMD:C_0402_1005Metric"
 			(at 37.7952 95.25 0)
 			(hide yes)
@@
 			)
 		)
-		(property "Footprint" "D8"
+		(property "Footprint" "OPA695:D8"
 			(at 40.64 69.85 0)
 			(hide yes)
@@
 			)
 		)
-		(property "Footprint" "ADE1"
+		(property "Footprint" "ADE-1+:ADE1"
 			(at 86.36 262.56 0)
 			(hide yes)
@@
 			)
 		)
-		(property "Footprint" "DSG0008A"
+		(property "Footprint" "OPA858:DSG0008A"
 			(at 232.41 36.83 0)
 			(hide yes)
@@
 	)
 	(symbol
+		(lib_id "Connector:TestPoint")
+		(at 166.37 182.88 0)
+		(unit 1)
+		(body_style 1)
+		(exclude_from_sim no)
+		(in_bom yes)
+		(on_board yes)
+		(in_pos_files yes)
+		(dnp no)
+		(fields_autoplaced yes)
+		(property "Reference" "TP1"
+			(at 168.91 178.3079 0)
+			(show_name no)
+			(do_not_autoplace no)
+			(effects
+				(font
+					(size 1.27 1.27)
+				)
+				(justify left)
+			)
+		)
+		(property "Value" "TestPoint"
+			(at 168.91 180.8479 0)
+			(show_name no)
+			(do_not_autoplace no)
+			(effects
+				(font
+					(size 1.27 1.27)
+				)
+				(justify left)
+			)
+		)
+		(property "Footprint" "TestPoint:TestPoint_Keystone_5015_Micro_Mini"
+			(at 171.45 182.88 0)
+			(hide yes)
+			(show_name no)
+			(do_not_autoplace no)
+			(effects
+				(font
+					(size 1.27 1.27)
+				)
+			)
+		)
+		(property "Datasheet" ""
+			(at 171.45 182.88 0)
+			(hide yes)
+			(show_name no)
+			(do_not_autoplace no)
+			(effects
+				(font
+					(size 1.27 1.27)
+				)
+			)
+		)
+		(property "Description" "test point"
+			(at 166.37 182.88 0)
+			(hide yes)
+			(show_name no)
+			(do_not_autoplace no)
+			(effects
+				(font
+					(size 1.27 1.27)
+				)
+			)
+		)
+		(pin "1"
+		)
+		(instances
+			(project "mts-demod"
+				(path "/6eb90501-7697-4fa3-aaec-602e91aa8771"
+					(reference "TP1")
+					(unit 1)
+				)
+			)
+		)
+	)
+	(symbol
 		(lib_id "power:GND")
 		(at 38.1 49.53 180)
@@
 			)
 		)
-		(property "Footprint" "CONN_SD-43045-005_08_MOL"
+		(property "Footprint" "430450812:CONN_SD-43045-005_08_MOL"
 			(at 113.03 170.18 0)
 			(hide yes)
@@
 			)
 		)
-		(property "Footprint" ""
+		(property "Footprint" "Inductor_SMD:L_0805_2012Metric"
 			(at 59.69 135.89 0)
 			(hide yes)
@@
 			)
 		)
-		(property "Footprint" ""
+		(property "Footprint" "TestPoint:TestPoint_Keystone_5015_Micro_Mini"
 			(at 265.43 31.75 0)
 			(hide yes)

Commit message: the most elegant board that i've ever laid out
Parts:
- added C40, C41: 0.1u, Capacitor_SMD:C_0603_1608Metric, symbol Device:C
- C19, C23, C24: footprint Capacitor_SMD:C_0805_2012Metric -> Capacitor_SMD:C_0402_1005Metric
- J3: value DEMOD INPUT -> RAW DEMOD ADC
Connections:
- net +5VA_GVA: now also C40.1, C41.1
- net GND: now also C40.2, C41.2
