File: mts-demod/.history/mts-demod.kicad_pcb (KiCad board)
At the start: 4 copper layers, 74.4 x 57.3 mm, 90 parts, among them IC1 ADE-1+, J1 RAW ERROR, J2 DEMOD IN, J3 DEMOD INPUT, J4 ANALOG ERROR, J5 PLP-5+, J6 INPUT PWR, U1 FDS010, U2 OPA858IDSGR, U3 OPA695IDR, U4 TCP-2-10X, U5 GVA-81, U6 0 dB atten, U7 PAT1220-C-4DB, U8 6 dB pad

Commit message: more Jack-ias
Routing:
- net GND: vias 518 -> 532
Changed lines of the file:
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@@
 		(tags "capacitor")
 		(property "Reference" "R15"
-			(at 3.105 -0.1 0)
+			(at 3.015 -1.31 0)
 			(layer "F.SilkS")
 			(effects
@@
 		(tags "capacitor")
 		(property "Reference" "C39"
-			(at 2.49 -0.02 90)
+			(at 2.96 0.01 90)
 			(layer "F.SilkS")
 			(effects
@@
 		(tags "capacitor")
 		(property "Reference" "R14"
-			(at 3.035 -0.03 0)
+			(at 3.035 -0.86 0)
 			(layer "F.SilkS")
 			(effects
@@
 	)
 	(via
+		(at 196.133347 76.57)
+		(size 0.6)
+		(drill 0.3)
+		(layers "F.Cu" "B.Cu")
+		(free yes)
+		(net "GND")
+	)
+	(via
 		(at 170.446274 88.298933)
 		(size 0.6)
@@
 	)
 	(via
+		(at 193.78 57.91)
+		(size 0.6)
+		(drill 0.3)
+		(layers "F.Cu" "B.Cu")
+		(free yes)
+		(net "GND")
+	)
+	(via
 		(at 156.15543 48.996705)
 		(size 0.6)
@@
 	)
 	(via
+		(at 174.12 86.36)
+		(size 0.6)
+		(drill 0.3)
+		(layers "F.Cu" "B.Cu")
+		(free yes)
+		(net "GND")
+	)
+	(via
 		(at 146.975 50.496875)
 		(size 0.6)
@@
 	)
 	(via
+		(at 193.46 60.73)
+		(size 0.6)
+		(drill 0.3)
+		(layers "F.Cu" "B.Cu")
+		(free yes)
+		(net "GND")
+	)
+	(via
 		(at 144.885118 69.45387)
 		(size 0.6)
@@
 	)
 	(via
+		(at 196.131155 74.945)
+		(size 0.6)
+		(drill 0.3)
+		(layers "F.Cu" "B.Cu")
+		(free yes)
+		(net "GND")
+	)
+	(via
 		(at 167.975 44.398784)
 		(size 0.6)
@@
 	)
 	(via
+		(at 193.85 55.27)
+		(size 0.6)
+		(drill 0.3)
+		(layers "F.Cu" "B.Cu")
+		(free yes)
+		(net "GND")
+	)
+	(via
 		(at 196.175 50.725)
 		(size 0.6)
@@
 	)
 	(via
+		(at 175.17 45.97)
+		(size 0.6)
+		(drill 0.3)
+		(layers "F.Cu" "B.Cu")
+		(free yes)
+		(net "GND")
+	)
+	(via
 		(at 140.252047 62.675)
 		(size 0.6)
@@
 	)
 	(via
+		(at 173.26 86.36)
+		(size 0.6)
+		(drill 0.3)
+		(layers "F.Cu" "B.Cu")
+		(free yes)
+		(net "GND")
+	)
+	(via
 		(at 163.15 44.400756)
 		(size 0.6)
@@
 	)
 	(via
+		(at 171.09 95.02)
+		(size 0.6)
+		(drill 0.3)
+		(layers "F.Cu" "B.Cu")
+		(free yes)
+		(net "GND")
+	)
+	(via
 		(at 128.532362 53.45)
 		(size 0.6)
@@
 	)
 	(via
+		(at 196.13 70.32)
+		(size 0.6)
+		(drill 0.3)
+		(layers "F.Cu" "B.Cu")
+		(free yes)
+		(net "GND")
+	)
+	(via
 		(at 152.346496 90.216792)
 		(size 0.6)
@@
 	)
 	(via
+		(at 173.95 42.99)
+		(size 0.6)
+		(drill 0.3)
+		(layers "F.Cu" "B.Cu")
+		(free yes)
+		(net "GND")
+	)
+	(via
 		(at 133.875 63.6)
 		(size 0.6)
@@
 	)
 	(via
+		(at 196.128431 73.40043)
+		(size 0.6)
+		(drill 0.3)
+		(layers "F.Cu" "B.Cu")
+		(free yes)
+		(net "GND")
+	)
+	(via
 		(at 151.57758 44.4)
 		(size 0.6)
@@
 	)
 	(via
+		(at 193.49 62.7)
+		(size 0.6)
+		(drill 0.3)
+		(layers "F.Cu" "B.Cu")
+		(free yes)
+		(net "GND")
+	)
+	(via
 		(at 151.575699 52.098261)
 		(size 0.6)
@@
 		(size 0.6)
 		(drill 0.3)
+		(layers "F.Cu" "B.Cu")
+		(free yes)
+		(net "GND")
+	)
+	(via
+		(at 196.13 71.82)
+		(size 0.6)
+		(drill 0.3)
