File: mts-clk/mts-clk.kicad_pcb (KiCad board)
At the start: 4 copper layers, 60.2 x 77.5 mm, 76 parts, among them IC1 SCPHS-13.6+, J1 Input (SMA), J2 Output (SMA), J3 Output (SMA), J4 Power Conn., J5 S2B-PH-K-SLFSN, U1 TCP-2-10X, U2 LTC6433BIUF-15-TRPBF, U3 LTC6433BIUF-15-TRPBF, U4 OPA197xD

Commit message: Jack's three vias
Routing:
- net GND: track 15.8 -> 17.6 mm, vias 428 -> 431
Changed lines of the file:
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@@
 		(capping no)
 		(filling no)
-		(zone_defaults)
 		(pcbplotparams
 			(layerselection 0x00000000_00000000_55555555_5755f5ff)
@@
 		(tags "capacitor")
 		(property "Reference" "C5"
-			(at -1.63 0.02 180)
+			(at -2.18 0.03 180)
 			(layer "F.SilkS")
 			(effects
@@
 	)
 	(segment
+		(start 146.46 88.53)
+		(end 146.46 89.29)
+		(width 0.2)
+		(layer "F.Cu")
+		(net "GND")
+	)
+	(segment
 		(start 126.61 116.309999)
 		(end 127.350001 116.309999)
@@
 	)
 	(segment
+		(start 148.85 81.87)
+		(end 149.28 82.75)
+		(width 0.2)
+		(layer "F.Cu")
+		(net "GND")
+	)
+	(segment
 		(start 160.975 93.28)
 		(end 160.975 94.35)
@@
 	)
 	(segment
+		(start 146.46 89.29)
+		(end 146.5 89.33)
+		(width 0.2)
+		(layer "F.Cu")
+		(net "GND")
+	)
+	(segment
 		(start 128.74 103.96)
 		(end 128.85 104.07)
@@
 	)
 	(via
+		(at 167.74 115.73)
+		(size 0.6)
+		(drill 0.3)
+		(layers "F.Cu" "B.Cu")
+		(net "GND")
+	)
+	(via
 		(at 136.005 87.685)
 		(size 0.6)
@@
 	)
 	(via
+		(at 146.46 88.53)
+		(size 0.6)
+		(drill 0.3)
+		(layers "F.Cu" "B.Cu")
+		(free yes)
+		(net "GND")
+	)
+	(via
 		(at 162.685 74.175)
 		(size 0.6)
@@
 	)
 	(via
+		(at 172.5 110.67)
+		(size 0.6)
+		(drill 0.3)
+		(layers "F.Cu" "B.Cu")
+		(free yes)
+		(net "GND")
+	)
+	(via
 		(at 158.63 74.175)
 		(size 0.6)
@@
 			)
 		)
+	)
+	(zone
+		(layer "F.Cu")
+		(hatch edge 0.5)
+		(connect_pads
+			(clearance 0)
+		)
+		(min_thickness 0.25)
+		(keepout
+			(tracks allowed)
+			(vias allowed)
+			(pads allowed)
+			(copperpour not_allowed)
+			(footprints allowed)
+		)
+		(placement
+			(enabled no)
+			(sheetname "")
+		)
+		(fill
+			(thermal_gap 0.5)
+			(thermal_bridge_width 0.5)
+			(island_removal_mode 0)
+		)
+		(polygon
+			(pts
+				(xy 128.26 118.55) (xy 128.832203 118.58) (xy 128.67 117.63) (xy 127.7 117.75) (xy 127.76 118.110002)
+			)
+		)
