File: mts-clk/mts-clk.kicad_sch (KiCad schematic)
At the start: 63 parts, among them IC1 SCPHS-13.6+, J1 Input (SMA), J2 Output (SMA), J3 Output (SMA), J4 Power Conn., J5 S2B-PH-K-SLFSN, U1 TCP-2-10X, U2 LTC6433BIUF-15-TRPBF, U3 LTC6433BIUF-15-TRPBF, U4 OPA197xD

Commit message: fixed atten issue
Connections:
- net 10MHz_DEMOD: now also R18.2, R19.1
- net 10MHz_EOM: no longer R18.2, R19.1
- net PORT1_POST_amp: no longer R17.1, R18.1
- net PORT2_POST_amp: now also R17.1, R18.1
Other:
- note added: "DEMOD path atten (7 dB)"

Commit message: final changes to CLK sch
Parts:
- added C29, C30: 0.1u, Capacitor_SMD:C_0603_1608Metric, symbol Device:C
- added C31: 22u, Capacitor_SMD:C_1206_3216Metric, symbol Device:C
- added C32, C34: 1u, Capacitor_SMD:C_0603_1608Metric, symbol Device:C
- added C33: 4.7u, Capacitor_SMD:C_1206_3216Metric, symbol Device:C
- added TP3: CONTROL TP, TestPoint:TestPoint_Keystone_5015_Micro_Mini, symbol Connector:TestPoint
- added TP4: PWM TP, TestPoint:TestPoint_Keystone_5015_Micro_Mini, symbol Connector:TestPoint
- IC1: footprint SCPHS136 -> SCPHS-13.6+:SCPHS136
- J1, J2, J3: footprint (none) -> SMA-J-P-H-ST-TH1:CONN_SMA-J-P-H-ST-TH1_SAI
- J4: footprint CONN_SD-43045-005_06_MOL -> 43045-005-06:CONN_SD-43045-005_06_MOL
- J5: footprint CONN_S2B-PH-K-S_JST -> S2B-PH-K-SLFSN:CONN_S2B-PH-K-S_JST
- L1, L3: footprint (none) -> Inductor_SMD:L_Coilcraft_LPS5030
- L2, L4: footprint (none) -> Inductor_SMD:L_0603_1608Metric
- R1: footprint (none) -> Resistor_SMD:R_0603_1608Metric
- R10, R8: value 81 -> 83.5
- R17, R19: value 131 -> 150
- R18: value 44.8 -> 37.4
- R9: value 100 -> 93.1
- U2, U3: footprint UF_24_ADI -> LTC6433:UF_24_ADI
Connections:
- net DGND is gone; now on net GND: J5.2
- net +15V: now also C33.1, C34.1
- net +5V: now also C29.2, C30.2, C31.2, C32.2
- net GND: now also C29.1, C30.1, C31.1, C32.1, C33.2, C34.2
- net V_CONTROL: now also TP3.1
- net V_FPGA_PWM: now also TP4.1
Other:
- note added: "DEMOD path atten (6 dB)"
- note added: "EOM path atten (12 dB)"
- note removed: "DEMOD path atten (7 dB)"
- note removed: "EOM path atten (12.5 dB)"
- moved on the sheet: J4, J5

Commit message: layout for CLK
Connections:
- net GND: now also IC1.12 (GROUND_8), IC1.13 (GROUND_9), IC1.14 (GROUND_10)
Changed lines of the file:
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@@
 	)
 	(junction
+		(at 219.71 93.98)
+		(diameter 0)
+		(color 0 0 0 0)
+	)
+	(junction
 		(at 50.8 171.45)
 		(diameter 0)
@@
 					(unit 1)
 				)
+			)
+		)
+	)
+	(symbol
+		(lib_id "power:GND")
+		(at 219.71 93.98 90)
+		(unit 1)
+		(body_style 1)
+		(exclude_from_sim no)
+		(in_bom yes)
+		(on_board yes)
+		(in_pos_files yes)
+		(dnp no)
+		(fields_autoplaced yes)
+		(property "Reference" "#PWR047"
+			(at 226.06 93.98 0)
+			(hide yes)
+			(show_name no)
+			(do_not_autoplace no)
+			(effects
+				(font
+					(size 1.27 1.27)
+				)
+			)
+		)
+		(property "Value" "GND"
+			(at 223.52 93.9799 90)
+			(show_name no)
+			(do_not_autoplace no)
+			(effects
+				(font
+					(size 1.27 1.27)
+				)
+				(justify right)
+			)
+		)
+		(property "Footprint" ""
+			(at 219.71 93.98 0)
+			(hide yes)
+			(show_name no)
+			(do_not_autoplace no)
+			(effects
+				(font
+					(size 1.27 1.27)
+				)
+			)
+		)
+		(property "Datasheet" ""
+			(at 219.71 93.98 0)
+			(hide yes)
+			(show_name no)
+			(do_not_autoplace no)
+			(effects
+				(font
+					(size 1.27 1.27)
+				)
+			)
+		)
+		(property "Description" "Power symbol creates a global label with name \"GND\" , ground"
+			(at 219.71 93.98 0)
+			(hide yes)
+			(show_name no)
+			(do_not_autoplace no)
+			(effects
+				(font
+					(size 1.27 1.27)
+				)
+			)
+		)
+		(pin "1"
+		)
+		(instances
+			(project "mts-clk"
+				(path "/70ecd414-537c-45a9-a21d-8f6fd964de4b"
+					(reference "#PWR047")
+					(unit 1)
+				)

Commit message: Jack's three vias
Parts:
- C4: value 1n -> 1nF
Changed lines of the file:
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@@
 			)
 		)
-		(property "Value" "1n"
+		(property "Value" "1nF"
 			(at 145.542 51.562 0)
 			(show_name no)
